File: Hardware/Power_Board.brd (EAGLE design)
At the start: 160 x 100 mm, 40 parts, among them K1 E3206S, K2 E3206S, K3 E3206S, K4 E3206S, K5 E3206S, K6 E3206S, Q1 BD135, Q2 BD135, Q3 BD135, Q4 BD135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

Commit message: Added a fuse to the power board and made PCB routes thicker.
Parts:
- added F1: 250V 2A, fuse:GSH15
- moved U$1 7.73 mm to (47.0, 66.0)
Connections:
- new net N$29: F1.2, U$1.LIVE
- net N$10: now also F1.1; no longer U$1.LIVE
Routing:
- net N$27: track 65.9 -> 120.3 mm
- net N$25: track 75.4 -> 94.4 mm
- net N$29: track 0.00 -> 18.5 mm
- net GND: track 347.4 -> 329.7 mm
- net N$10: track 112.4 -> 94.9 mm
- net N$8: track 75.1 -> 87.1 mm
- net N$1: track 69.4 -> 79.2 mm
- net VCC: track 274.2 -> 265.9 mm
- net PIN4: track 60.7 -> 64.7 mm
- net N$28: track 65.2 -> 64.1 mm
- net N$26: track 65.6 -> 66.4 mm
- net N$23: track 94.8 -> 95.4 mm
